File: STM32F4Stick.brd (EAGLE design)
At the start: 46.7 x 25.9 mm, 46 parts, among them U1 MIC5219 3.3V, U2 USD-SOCKETNEW

Commit message: button fix
Connections:
- net BOOT1: no longer S2.3
- net GND: no longer S1.2
- net NRST: no longer S1.3
- net VCC: no longer S2.2
Routing:
- net NRST: track 18.6 -> 20.7 mm
- net GND: track 40.9 -> 38.8 mm
- net BOOT1: track 24.4 -> 25.7 mm
Changed lines of the file:
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@@
 <text x="11.176" y="4.826" size="0.4064" layer="21">JTMS</text>
 <text x="13.716" y="4.826" size="0.4064" layer="21">JTCK</text>
-<text x="16.51" y="4.064" size="0.4064" layer="21" ratio="15">JTDI</text>
+<text x="16.51" y="4.064" size="0.4064" layer="21" ratio="7">JTDI</text>
 <text x="29.464" y="4.064" size="0.4064" layer="21">JTD0</text>
 <text x="31.496" y="4.064" size="0.4064" layer="21">NJTRST</text>
@@
 <text x="25.654" y="16.764" size="0.3048" layer="22" font="vector" rot="MR0">For STM32F401
 0-ohm res</text>
+<rectangle x1="0.254" y1="23.114" x2="3.302" y2="25.654" layer="21"/>
 </plain>
 <attributes>
@@
 <wire x1="31.496" y1="19.558" x2="38.354" y2="19.558" width="0.254" layer="16"/>
 <wire x1="38.354" y1="19.558" x2="38.862" y2="19.558" width="0.254" layer="1"/>
-<wire x1="38.862" y1="19.558" x2="41.656" y2="16.764" width="0.254" layer="1"/>
-<wire x1="41.656" y1="16.764" x2="42.418" y2="16.764" width="0.254" layer="1"/>
-<wire x1="42.418" y1="16.764" x2="45.466" y2="16.764" width="0.254" layer="1"/>
-<wire x1="45.466" y1="16.764" x2="45.974" y2="16.256" width="0.254" layer="1"/>
-<wire x1="45.974" y1="16.256" x2="45.974" y2="11.684" width="0.254" layer="1"/>
+<wire x1="45.974" y1="15.748" x2="45.974" y2="11.684" width="0.254" layer="1"/>
 <wire x1="45.974" y1="11.684" x2="44.958" y2="10.668" width="0.254" layer="1"/>
 <wire x1="44.958" y1="10.668" x2="43.434" y2="10.668" width="0.254" layer="1"/>
@@
 <wire x1="12.192" y1="24.384" x2="13.462" y2="23.114" width="0.2032" layer="1"/>
 <wire x1="13.462" y1="23.114" x2="13.462" y2="19.812" width="0.2032" layer="1"/>
-<contactref element="S2" pad="2"/>
+<wire x1="38.862" y1="19.558" x2="41.91" y2="16.764" width="0.254" layer="1"/>
+<wire x1="41.91" y1="16.764" x2="42.566" y2="16.764" width="0.254" layer="1"/>
+<wire x1="42.566" y1="16.764" x2="42.588" y2="16.742" width="0.254" layer="1"/>
+<wire x1="45.974" y1="15.748" x2="43.836" y2="15.748" width="0.254" layer="1"/>
+<wire x1="43.836" y1="15.748" x2="42.588" y2="16.742" width="0.254" layer="1"/>
 </signal>
 <signal name="GND">
@@
 <wire x1="44.45" y1="11.938" x2="44.45" y2="12.839" width="0.2032" layer="1"/>
 <wire x1="44.45" y1="12.839" x2="44.565" y2="13.208" width="0.2032" layer="1"/>
-<wire x1="41.148" y1="5.334" x2="42.312" y2="5.334" width="0.2032" layer="1"/>
 <wire x1="42.312" y1="5.334" x2="42.334" y2="5.312" width="0.2032" layer="1"/>
-<wire x1="42.356" y1="5.334" x2="44.45" y2="5.334" width="0.2032" layer="1"/>
 <wire x1="42.356" y1="5.334" x2="42.334" y2="5.312" width="0.2032" layer="1"/>
 <polygon width="0.2032" layer="1" isolate="0.3048">
@@
 <contactref element="C12" pad="2"/>
 <contactref element="C17" pad="2"/>
-<contactref element="S1" pad="2"/>
+<wire x1="41.148" y1="5.334" x2="42.334" y2="5.334" width="0.254" layer="1"/>
+<wire x1="42.334" y1="5.334" x2="42.334" y2="5.312" width="0.254" layer="1"/>
 </signal>
 <signal name="N$10">
@@
 <wire x1="31.75" y1="12.7" x2="37.338" y2="11.938" width="0.2032" layer="16"/>
 <via x="37.338" y="11.938" extent="1-16" drill="0.4064"/>
-<wire x1="42.338" y1="8.978" x2="42.334" y2="8.974" width="0.2032" layer="1"/>
 <wire x1="28.79" y1="12.7" x2="31.75" y2="12.7" width="0.254" layer="16"/>
-<wire x1="41.822" y1="8.978" x2="37.338" y2="11.938" width="0.254" layer="1"/>
-<wire x1="44.534" y1="8.912" x2="42.396" y2="8.912" width="0.2032" layer="1"/>
-<wire x1="42.396" y1="8.912" x2="42.334" y2="8.974" width="0.2032" layer="1"/>
-<wire x1="41.822" y1="8.978" x2="42.33" y2="8.978" width="0.254" layer="1"/>
-<wire x1="42.33" y1="8.978" x2="42.334" y2="8.974" width="0.254" layer="1"/>
-<contactref element="S1" pad="3"/>
+<wire x1="44.534" y1="8.912" x2="44.534" y2="8.466" width="0.254" layer="1"/>
+<wire x1="44.534" y1="8.466" x2="43.434" y2="7.366" width="0.254" layer="1"/>
+<wire x1="43.434" y1="7.366" x2="41.148" y2="7.366" width="0.254" layer="1"/>
+<wire x1="41.148" y1="7.366" x2="37.338" y2="11.938" width="0.254" layer="1"/>
 </signal>
 <signal name="USB_DP">
@@
 <wire x1="24.638" y1="20.408" x2="35.902" y2="20.408" width="0.2032" layer="16"/>
 <wire x1="35.902" y1="20.408" x2="36.068" y2="20.574" width="0.254" layer="16"/>
-<wire x1="44.788" y1="20.342" x2="36.3" y2="20.342" width="0.2032" layer="1"/>
 <wire x1="36.3" y1="20.342" x2="36.068" y2="20.574" width="0.2032" layer="1"/>
-<contactref element="S2" pad="3"/>
+<wire x1="36.3" y1="20.342" x2="40.11" y2="20.342" width="0.254" layer="1"/>
+<wire x1="40.11" y1="20.342" x2="41.402" y2="19.05" width="0.254" layer="1"/>
+<wire x1="41.402" y1="19.05" x2="43.688" y2="19.05" width="0.254" layer="1"/>
+<wire x1="43.688" y1="19.05" x2="44.704" y2="20.32" width="0.254" layer="1"/>
+<wire x1="44.704" y1="20.32" x2="44.704" y2="20.258" width="0.254" layer="1"/>
+<wire x1="44.704" y1="20.258" x2="44.788" y2="20.342" width="0.254" layer="1"/>
 </signal>
 <signal name="5V">
